File: 02_Estacion/Hardware/V2_Estacion_Nivel/V2_Estacion_Nviel.kicad_pcb (KiCad board)
At the start: 2 copper layers, 100 x 100 mm, 62 parts, among them J1 Micro_SD_Card_Det1, J3 Screw_Terminal_01x02, J4 Screw_Terminal_01x02, J5 Screw_Terminal_01x02, J6 Conn_01x10_Pin, J7 Conn_01x02_Pin, J8 Screw_Terminal_01x04, J9 USB_C_Receptacle_USB2.0_16P, SW1 RST, SW2 BOOT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

Commit message: commit
Parts:
- moved C14 8.56 mm to (150.9, 43.0)
- moved R12 8.21 mm to (150.8, 48.0)
- moved C10 7.57 mm to (156.9, 43.0)
- moved C11 7.22 mm to (156.9, 48.0)
- moved U2 7.16 mm to (170.1, 49.8)
- moved C12 7.15 mm to (142.8, 50.0)
- moved C13 7.15 mm to (133.8, 50.0)
- moved SW1 7.15 mm to (142.8, 43.8)
- moved SW2 7.15 mm to (133.8, 43.8)
- moved D8 2.24 mm to (105.0, 96.0)
- moved G*** 2.24 mm to (119.0, 53.0)
- moved R15 2.00 mm to (114.0, 89.0)
- moved D2 1.40 mm to (160.6, 66.0)
- moved D6 1.40 mm to (160.6, 71.0)
- moved D7 1.40 mm to (160.6, 76.0)
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Routing:
- net 3V3: track 446.6 -> 467.4 mm
- net GND: track 7.78 -> 16.7 mm, vias 5 -> 6
- net Net-(D7-A): track 0.00 -> 8.24 mm
- net DE/RE 1: track 85.9 -> 93.5 mm
- net DE/RE 2: track 94.3 -> 87.1 mm, vias 4 -> 2
- net D+: track 79.8 -> 72.6 mm, vias 3 -> 2
- net RO2: track 71.9 -> 79.1 mm
- net D-: track 79.9 -> 72.8 mm, vias 4 -> 3
- net SQW: track 74.1 -> 67.1 mm
- net Net-(D6-A): track 0.00 -> 6.85 mm
- net GPIO38: track 26.1 -> 32.6 mm
- net SDA: track 64.8 -> 58.3 mm
- net VCC: track 157.1 -> 163.5 mm
- net GPIO39: track 24.9 -> 31.0 mm
- net GPIO41: track 22.3 -> 28.3 mm
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
Commit message: commit
Routing:
- net GND: track 16.7 -> 23.8 mm, vias 6 -> 7
Changed lines of the file:
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@@
 		(tags "capacitor handsolder")
 		(property "Reference" "C5"
-			(at -4.2125 0 0)
+			(at -3.2125 1 0)
 			(layer "F.SilkS")
 			(effects
@@
 	)
 	(segment
+		(start 126 121)
+		(end 125 120)
+		(width 0.25)
+		(layer "F.Cu")
+		(net 1)
+	)
+	(segment
 		(start 182.25 95.25)
 		(end 183 96)
@@
 	)
 	(segment
+		(start 125 120)
+		(end 123.825 120)
+		(width 0.25)
+		(layer "F.Cu")
+		(net 1)
+	)
+	(segment
 		(start 167.2 49.2)
 		(end 167.01 49.2)
@@
 	)
 	(segment
-		(start 127.43 102.43)
-		(end 127 102)
+		(start 126 103.7)
+		(end 126 103)
+		(width 0.25)
+		(layer "F.Cu")
+		(net 1)
+	)
+	(segment
+		(start 126 105)
+		(end 125 106)
 		(width 0.25)
 		(layer "F.Cu")
@@
 	)
 	(segment
+		(start 126.57 102.43)
+		(end 128.7 102.43)
+		(width 0.25)
+		(layer "F.Cu")
+		(net 1)
+	)
+	(segment
 		(start 100.94 90.09)
 		(end 101.09 90.09)
@@
 	)
 	(segment
-		(start 155 48)
-		(end 154 47)
+		(start 126 103)
+		(end 126.57 102.43)
 		(width 0.25)
 		(layer "F.Cu")
@@
 	)
 	(segment
-		(start 128.7 102.43)
-		(end 127.43 102.43)
+		(start 155 48)
+		(end 154 47)
 		(width 0.25)
 		(layer "F.Cu")
@@
 		(net 1)
 	)
+	(segment
+		(start 126 103.7)
+		(end 126 105)
+		(width 0.25)
+		(layer "F.Cu")
+		(net 1)
+	)
 	(via
-		(at 172 49)
+		(at 125 106)
 		(size 0.6)
 		(drill 0.3)
@@
 	)
 	(via
-		(at 167 133)
+		(at 126 121)
 		(size 0.6)
 		(drill 0.3)
@@
 	)
 	(via
-		(at 127 102)
+		(at 172 49)
+		(size 0.6)
+		(drill 0.3)
+		(layers "F.Cu" "B.Cu")
+		(net 1)
+	)
+	(via
+		(at 167 133)
 		(size 0.6)
 		(drill 0.3)
@@
 	)
 	(segment
-		(start 179.39219 44.03)
-		(end 179.926 44.56381)
-		(width 0.25)
-		(layer "F.Cu")
-		(net 26)
-	)
-	(segment
 		(start 183.4925 89.345)
 		(end 184 88.8375)
@@
 	)
 	(segment
-		(start 179.926 44.926)
-		(end 192.92 57.92)
+		(start 179.39219 44.03)
+		(end 179.926 44.56381)
 		(width 0.25)
 		(layer "F.Cu")
@@
 	)
 	(segment
-		(start 192.92 57.92)
-		(end 195 57.92)
+		(start 179.926 44.926)
+		(end 192.92 57.92)
 		(width 0.25)
 		(layer "F.Cu")
@@
 	)
 	(segment
-		(start 194.92 57.92)
+		(start 192.92 57.92)
 		(end 195 57.92)
 		(width 0.25)
@@
 		(width 0.25)
 		(layer "F.Cu")
+		(net 26)
+	)
+	(segment
+		(start 194.92 57.92)
+		(end 195 57.92)
+		(width 0.25)
+		(layer "F.Cu")

Commit message: commit
Routing:
- net SDA: track 58.3 -> 59.5 mm
Changed lines of the file:
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@@
+	)
+	(segment
+		(start 143.85 50)
+		(end 144.85 50)
+		(width 0.25)
+		(layer "F.Cu")
+		(net 4)
 	)
 	(segment
@@
 	)
 	(segment
+		(start 146.85 48)
+		(end 146.85 45)
+		(width 0.25)
+		(layer "F.Cu")
+		(net 4)
+	)
+	(segment
 		(start 152.85 50)
 		(end 156.85 50)
@@
 	)
 	(segment
+		(start 144.85 50)
+		(end 146.85 48)
+		(width 0.25)
+		(layer "F.Cu")
+		(net 4)
+	)
+	(segment
 		(start 156.85 50)
 		(end 157.925 48.925)
@@
 	(segment
 		(start 143.85 50)
-		(end 144.85 50)
-		(width 0.25)
-		(layer "F.Cu")
-		(net 4)
-	)
-	(segment
-		(start 143.85 50)
 		(end 149.85 50)
-		(width 0.25)
-		(layer "F.Cu")
-		(net 4)
-	)
-	(segment
-		(start 144.85 50)
-		(end 146.85 48)
 		(width 0.25)
 		(layer "F.Cu")
@@
 	)
 	(segment
-		(start 146.85 48)
-		(end 146.85 45)
-		(width 0.25)
-		(layer "F.Cu")
-		(net 4)
-	)
-	(segment
 		(start 139 67.6)
 		(end 139 49.15)
@@
 	)
 	(segment
-		(start 131.14 73.54)
-		(end 103 73.54)
-		(width 0.25)
-		(layer "F.Cu")
-		(net 31)
-	)
-	(segment
 		(start 153.55 73)
 		(end 152.6 73)
@@
 	)
 	(segment
+		(start 125 73.54)
+		(end 103 73.54)
+		(width 0.25)
+		(layer "F.Cu")
+		(net 31)
+	)
+	(segment
 		(start 167 73)
 		(end 173.275 66.725)
@@
 	)
 	(via
-		(at 131.14 73.54)
+		(at 125 73.54)
 		(size 0.6)
 		(drill 0.3)
@@
 	)
 	(segment
-		(start 132.6 73)
-		(end 152.6 73)
+		(start 125.54 73)
+		(end 125 73.54)
 		(width 0.25)
 		(layer "B.Cu")
@@
 	)
 	(segment
-		(start 132.06 73.54)
-		(end 132.6 73)
-		(width 0.25)
-		(layer "B.Cu")
-		(net 31)
-	)
-	(segment
-		(start 131.14 73.54)
-		(end 132.06 73.54)
+		(start 152.6 73)
+		(end 125.54 73)
 		(width 0.25)
 		(layer "B.Cu")
@@
 	)
 	(segment
-		(start 161.35 55.46)
-		(end 159.654702 55.46)
-		(width 0.25)
-		(layer "F.Cu")
-		(net 43)
-	)
-	(segment
-		(start 159.654702 55.46)
-		(end 137 78.114702)
+		(start 137 76)
+		(end 137 93)
 		(width 0.25)
 		(layer "F.Cu")
@@
 	)
 	(segment
+		(start 157.54 55.46)
+		(end 137 76)
+		(width 0.25)
+		(layer "F.Cu")
+		(net 43)
+	)
+	(segment
 		(start 139.38 98.62)
 		(end 138 98.62)
@@
 	)
 	(segment
-		(start 137 78.114702)
-		(end 137 93)
-		(width 0.25)
-		(layer "F.Cu")
-		(net 43)
-	)
-	(segment
 		(start 137 93)
 		(end 139 93)
 		(width 0.25)
 		(layer "F.Cu")
+		(net 43)
+	)
+	(segment
+		(start 161.35 55.46)
+		(end 157.54 55.46)
+		(width 0.25)
+		(layer "F.Cu")
