File: 02_Estacion/Proyecto3__Sistema_de_adquisiscion_de_Nivel/Hardware_Kicad/V1_Estacion_Nivel/Estacion_Nivel.kicad_pcb (KiCad board)
At the start: 4 copper layers, 100 x 100 mm, 61 parts, among them J1 503398-1892, J10 M20-9991045, J2 1751248, J3 1751248, J4 1751248, J5 1751248, J7 M20-9990245, J8 RASM722PTR13X, J9 USB4085-GF-A_REVA4, SW1 RST, SW2 BOOT, U1 SP3485EN-L_TR, U2 ESP32-S3-WROOM-1-N16R8, U3 LM1117MPX-3.3_NOPB, U4 DS3231MZ+, U5 SP3485EN-L_TR

Commit message: update
Routing:
- net GND: track 161.7 -> 160.9 mm, vias 45 -> 46
Changed lines of the file:
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@@
 			(crossoutdnponfab yes)
 			(subtractmaskfromsilk no)
-			(outputformat 1)
+			(outputformat 5)
 			(mirror no)
-			(drillshape 1)
+			(drillshape 0)
 			(scaleselection 1)
 			(outputdirectory "")
@@
 	)
 	(gr_text "${REFERENCE}"
-		(at 125.3 46.5 0)
+		(at 109 36 0)
 		(layer "F.Fab")
 		(effects
@@
 	)
 	(segment
+		(start 136.925 35.925)
+		(end 136 35)
+		(width 0.5)
+		(layer "F.Cu")
+		(net 1)
+	)
+	(segment
 		(start 180.6 89)
 		(end 180.6 91.1)
@@
 	)
 	(segment
+		(start 136.925 39.06)
+		(end 136.925 35.925)
+		(width 0.5)
+		(layer "F.Cu")
+		(net 1)
+	)
+	(segment
 		(start 192.725 101.115)
 		(end 192.725 99.775)
@@
 	)
 	(via
+		(at 136 35)
+		(size 0.6)
+		(drill 0.3)
+		(layers "F.Cu" "B.Cu")
+		(net 1)
+	)
+	(via
 		(at 178.525 104.475)
 		(size 0.6)
@@
 		(net 1)
 	)
-	(segment
-		(start 107.5 65.44)
-		(end 111.2 69.14)
-		(width 0.5)
-		(layer "In1.Cu")
-		(net 1)
-	)
