File: 02_Estacion/Proyecto3__Sistema_de_adquisiscion_de_Nivel/Hardware_Kicad/V2_Estacion_Nivel/DS3231.kicad_sch (KiCad schematic)
At the start: 8 parts, among them U4 DS3231M

Commit message: update
Other:
- moved on the sheet: BT1, C6, C7, D3, R18, R19, R20, U4
