File: 02_Estacion/Proyecto3__Sistema_de_adquisiscion_de_Nivel/Hardware_Kicad/V2_Estacion_Nivel/ttl_to_rs485.kicad_sch (KiCad schematic)
At the start: 18 parts, among them J4 Screw_Terminal_01x02, J5 Screw_Terminal_01x02, U1 SP3485EN, U5 SP3485EN

Commit message: update
Other:
- moved on the sheet: C8, C9, D1, D5, J4, J5, R1, R17, R2, R22, R23, R24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
