File: 02_Estacion/Proyecto3__Sistema_de_adquisiscion_de_Nivel/Hardware_Kicad/V2_Estacion_Nivel/vcc_to_3v3.kicad_sch (KiCad schematic)
At the start: 5 parts, among them J3 Screw_Terminal_01x02, J8 Screw_Terminal_01x04, U3 AMS1117-3.3

Commit message: update
Other:
- moved on the sheet: C4, C5, J3, J8, U3
